File: test/common/resources/fileformats/kicad/v10/pcb/via_treatments.kicad_pcb (KiCad board)
At the start: 6 copper layers, 28 x 28 mm, 7 parts, among them P1 TestPoint_Pad_D2.0mm, P2 TestPoint_Pad_D2.0mm, P3 TestPoint_Pad_D2.0mm, P4 TestPoint_Pad_D2.0mm, P5 TestPoint_Pad_D2.0mm, P6 TestPoint_Pad_D2.0mm

Commit message: pad grammar closure: pressfit property, pad-level hole treatments, KiCad emission order
Three empirically reproduced burns against KiCad 10.0.3 ground truth
(pcb_io_kicad_sexpr[_parser].cpp), all in pcb.zig's Pad/Footprint:

1. CRITICAL: E_pad_property was missing pad_prop_pressfit. Since the
   in-range re-key of the field from 'properties' to 'property' made the
   enum path reachable, any v10 board with a press-fit pad hard-failed
   loads() with InvalidValue (board-blocking; before the re-key it was a
   warn+drop). Token added in the 10.0.3 writer position (after
   pad_prop_mechanical); the enum is now closed over all 9 tokens the
   writer emits.

2. MAJOR: Pad modeled none of backdrill / tertiary_drill /
   front_post_machining / back_post_machining although all four are
   pad-level in the 10.0.3 grammar (format(PAD) :1735-1777, parsePAD) —
   real counterbore/backdrill fabrication data was S5a-dropped on any
   managed rewrite. Added as optional fields reusing the existing
   Backdrill/PostMachining types.

3. MINOR: (property ...) was declared (= emitted) after thermal_gap;
   KiCad writes it after the post-machining slot and before (layers ...)
   — reorder churn on the first KiCad resave. Moved to the writer slot.
   Same class: net_tie_pad_groups now precedes
   duplicate_pad_numbers_are_jumpers (writer :1390 vs :1398).

Fixture: via_treatments.kicad_pcb gains a press-fit THT pad carrying all
four hole treatments; kicad-cli 10.0.3-normalized, drc rc==0 both as
committed and after our loads()->dumps() rewrite (empirically verified;
semantic snapshot regenerated — diff is purely the added footprint, via
net bindings unchanged).

Tests (test_padstack_dialect.py, +14): every writer property token loads
(param x9), pad hole-treatment roundtrip + no-data-loss, pad write order
vs format(PAD), footprint net_tie order, absent-treatments-stay-absent.
Mutation-verified: all five guards ran red against the pre-fix pcb.zig
(pressfit InvalidValue, treatments Attribu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
Parts:
- added P7: TestPoint_THTPad_D1.5mm_Drill0.7mm, TestPoint:TestPoint_THTPad_D1.5mm_Drill0.7mm, F.Cu at (122.0, 100.0)
